File: plate/plate.sch (KiCad schematic (older format))
At the start: 6 parts, among them J1 Conn_01x06, J2 Conn_01x06, J3 Conn_01x06, J4 Conn_01x06, J5 Conn_01x06, J6 Conn_01x06

Commit message: Use single IDC header and prep outline for magnets
Parts:
- J1, J2, J3, J4, J5, J6: footprint keyboard-parts:header_1x06_2.54mm -> keyboard-parts:header_sym_1x06_2.54mm
Changed lines of the file:
@@
 EESchema Schematic File Version 4
+LIBS:plate-cache
 EELAYER 30 0
 EELAYER END
@@
 F 0 "J1" H 1200 1500 50  0000 C CNN
 F 1 "Conn_01x06" H 1200 800 50  0000 C CNN
-F 2 "keyboard-parts:header_1x06_2.54mm" H 1200 1200 50  0001 C CNN
+F 2 "keyboard-parts:header_sym_1x06_2.54mm" H 1200 1200 50  0001 C CNN
 F 3 "~" H 1200 1200 50  0001 C CNN
 	1    1200 1200
@@
 F 0 "J2" H 1700 1500 50  0000 C CNN
 F 1 "Conn_01x06" H 1700 800 50  0000 C CNN
-F 2 "keyboard-parts:header_1x06_2.54mm" H 1700 1200 50  0001 C CNN
+F 2 "keyboard-parts:header_sym_1x06_2.54mm" H 1700 1200 50  0001 C CNN
 F 3 "~" H 1700 1200 50  0001 C CNN
 	1    1700 1200
@@
 F 0 "J3" H 2200 1500 50  0000 C CNN
 F 1 "Conn_01x06" H 2200 800 50  0000 C CNN
-F 2 "keyboard-parts:header_1x06_2.54mm" H 2200 1200 50  0001 C CNN
+F 2 "keyboard-parts:header_sym_1x06_2.54mm" H 2200 1200 50  0001 C CNN
 F 3 "~" H 2200 1200 50  0001 C CNN
 	1    2200 1200
@@
 F 0 "J4" H 2700 1500 50  0000 C CNN
 F 1 "Conn_01x06" H 2700 800 50  0000 C CNN
-F 2 "keyboard-parts:header_1x06_2.54mm" H 2700 1200 50  0001 C CNN
+F 2 "keyboard-parts:header_sym_1x06_2.54mm" H 2700 1200 50  0001 C CNN
 F 3 "~" H 2700 1200 50  0001 C CNN
 	1    2700 1200
@@
 F 0 "J5" H 3200 1500 50  0000 C CNN
 F 1 "Conn_01x06" H 3200 800 50  0000 C CNN
-F 2 "keyboard-parts:header_1x06_2.54mm" H 3200 1200 50  0001 C CNN
+F 2 "keyboard-parts:header_sym_1x06_2.54mm" H 3200 1200 50  0001 C CNN
 F 3 "~" H 3200 1200 50  0001 C CNN
 	1    3200 1200
@@
 F 0 "J6" H 3700 1500 50  0000 C CNN
 F 1 "Conn_01x06" H 3700 800 50  0000 C CNN
-F 2 "keyboard-parts:header_1x06_2.54mm" H 3700 1200 50  0001 C CNN
+F 2 "keyboard-parts:header_sym_1x06_2.54mm" H 3700 1200 50  0001 C CNN
 F 3 "~" H 3700 1200 50  0001 C CNN
 	1    3700 1200
