File: plate/plate.kicad_pcb (KiCad board)
At the start: 2 copper layers, 157.7 x 114.5 mm, 8 parts, among them J1 Conn_01x06, J2 Conn_01x06, J3 Conn_01x06, J4 Conn_01x06, J5 Conn_01x06, J6 Conn_01x06

Commit message: Update version number to v2 and add new gerbers
Other:
- outline, holes or cut-outs redrawn
- board text added: "Stomp v2"
- board text removed: "Stomp v1"
